Commit message: second commit

File: iter_1/jetchair_urdf/urdf/jetchair_urdf.urdf (robot description, URDF)
Before this commit: robot autochair, 6 links, 5 joints
Links:
- link base_link: mass 31.4560304030786 -> 31.4560304030766; geometry collision mesh filename=package://jetchair_urdf/meshes/base_link.STL; visual mesh filename=package://jetchair_urdf/meshes/base_link.STL
- link left_caster_wheel: mass 0.24268 -> 0.242680705446467; geometry collision mesh filename=package://jetchair_urdf/meshes/left_caster_wheel.STL; visual mesh filename=package://jetchair_urdf/meshes/left_caster_wheel.STL
- link left_wheel: geometry collision mesh filename=package://jetchair_urdf/meshes/left_wheel.STL; visual mesh filename=package://jetchair_urdf/meshes/left_wheel.STL
- link lidar: geometry collision mesh filename=package://jetchair_urdf/meshes/lidar.STL; visual mesh filename=package://jetchair_urdf/meshes/lidar.STL
- link right_caster_wheel: mass 0.24268 -> 0.242680594536878; geometry collision mesh filename=package://jetchair_urdf/meshes/right_caster_wheel.STL; visual mesh filename=package://jetchair_urdf/meshes/right_caster_wheel.STL
- link right_wheel: mass 1.8909 -> 1.89094567469007; geometry collision mesh filename=package://jetchair_urdf/meshes/right_wheel.STL; visual mesh filename=package://jetchair_urdf/meshes/right_wheel.STL
Joints:
- joint left_caster_joint: origin xyz=-2.3764 3.3374 0.12015 rpy=1.5708 0 0 -> xyz=-2.3763778140888 3.33736396242897 0.120147829114934 rpy=1.5707963267949 0 0
- joint left_wheel_joint: origin xyz=-2.9142 3.3404 0.044848 rpy=1.5708 0 0 -> xyz=-2.9141678140888 3.34036396242897 0.0448478291149333 rpy=1.5707963267949 0 0
- joint lidar_joint: origin xyz=-2.6586 3.1054 0.1445 rpy=1.5708 0 0 -> xyz=-2.65862808664732 3.10536396242897 0.144497829114934 rpy=1.5707963267949 0 0
- joint right_wheel_joint: origin xyz=-2.8933 3.1004 0.50776 rpy=1.5708 0 0 -> xyz=-2.89326802793966 3.10036396242897 0.507755393218783 rpy=1.5707963267949 0 0

Commit message: commit urdf

File: iter_1/jetchair_urdf/urdf/jetchair_urdf.urdf (robot description, URDF)
Before this commit: robot jetchair_urdf, 6 links, 5 joints
Links:
- link base_link: mass 31.4560304030766 -> 31.4560304041365
- link right_caster_wheel: mass 0.242680594536878 -> 0.242680594536877
Joints:
- joint right_wheel_joint: origin xyz=-2.89326802793966 3.10036396242897 0.507755393218783 rpy=1.5707963267949 0 0 -> xyz=-2.9141678140888 2.86036396242897 0.0448478291149336 rpy=1.5707963267949 0 0
